Commit message: fix math eval on property

File: examples/py/xacro/source_example/property.xacro (robot description, xacro)
@@ -5,5 +5,5 @@
         <visual>
             <geometry>
-                <cylinder radius="${width}" length="${bodylen}" />
+                <cylinder radius="${2*width}" length="${bodylen}" />
             </geometry>
             <material name="blue">

Commit message: subsitute node text

File: examples/py/xacro/source_example/property.xacro (robot description, xacro)
@@ -2,5 +2,9 @@
     <xacro:property name="width" value=".2" />
     <xacro:property name="bodylen" value=".6" />
+    <xacro:property name="x" value="1" />
+    <xacro:property name="y" value="2" />
+    <xacro:property name="z" value="3" />
     <link name="base_link">
+        <pose>${x} ${y} ${z} 0 0 0</pose>
         <visual>
             <geometry>
