Commit message: fix: remove xacro from sdf

File: examples/py/xacro/source_example/common.xacro (robot description, xacro)
@@ -12,3 +12,24 @@
     </inertia>
 </xacro:macro>
+<!-- inertia_cylinder -->
+<xacro:macro name="inertia_cylinder" params="m r l">
+    <mass>${m}</mass>
+    <inertia>
+        <ixx>${m*(3*r*r+l*l)/12}</ixx>
+        <ixy>0</ixy>
+        <ixz>0</ixz>
+        <iyy>${m*(3*r*r+l*l)/12}</iyy>
+        <iyz>0</iyz>
+        <izz>${m*r*r/2}</izz>
+    </inertia>
+</xacro:macro>
+<!-- geometry_cylinder -->
+<xacro:macro name="geometry_cylinder" params="r l">
+    <geometry>
+        <cylinder>
+            <radius>${r}</radius>
+            <length>${l}</length>
+        </cylinder>
+    </geometry>
+</xacro:macro>
 </sdf>

File: examples/py/xacro/source_example/data.xacro (robot description, xacro)
@@ -1,7 +1,10 @@
 <sdf xmlns:xacro="http://dd">
-    <xacro:property name="name" value="aaaa" />
+    <xacro:property name="base_mass" value="200" />
     <xacro:property name="bodylen" value=".6" />
     <xacro:property name="x" value="1" />
     <xacro:property name="y" value="2" />
     <xacro:property name="z" value="3" />
+    <xacro:property name="wheel_mass" value="2" />
+    <xacro:property name="wheel_r" value="0.5" />
+    <xacro:property name="wheel_l" value="0.1" />
 </sdf>

File: examples/py/xacro/source_example/macro.sdf.xacro (robot description, xacro)
@@ -1,6 +1,7 @@
-<sdf xmlns:xacro="http://dd">
+<sdf version="1.7" xmlns:xacro="http://dd">
     <xacro:include uri="file://data.xacro" />
     <xacro:include uri="file://common.xacro" />
-    <xacro:property name="base_mass" value="100" />
+    <xacro:include uri="file://color.xacro" />
+    <xacro:property name="base_mass2" value="100" />
     <model name='heavy_base'>
         <pose>0 0 0 0 0 0</pose>
@@ -9,5 +10,5 @@
             <pose>0 0 0.05 0 0 0</pose>
             <inertial>
-                <xacro:inertia_box m="100" x="2.2" y="1" z="0.1" />
+                <xacro:inertia_box m="${base_mass}" x="2.2" y="1" z="0.1" />
             </inertial>
             <!-- Same geometry as visual -->
@@ -33,4 +34,19 @@
             </visual>
         </link>
+        <link name="wheel_left">
+            <pose>0 -0.5 0 1.5707 0 0</pose>
+            <inertial>
+                <xacro:inertia_cylinder m="${wheel_mass}" r="${wheel_r}" l="${wheel_l}" />
+            </inertial>
+            <visual name="wheel_left_visual">
+                <xacro:geometry_cylinder r="${wheel_r}" l="${wheel_l}"/>
+                <material>
+                    <xacro:color color_name="Red"/>
+                </material>
+            </visual>
+            <collision name="wheel_left_collision">
+                <xacro:geometry_cylinder r="${wheel_r}" l="${wheel_l}"/>
+            </collision>
+        </link>
     </model>
 </sdf>
