Commit message: fix: macro
macro inner xml
macro eval
macro append to source

File: examples/py/xacro/source_example/macro.sdf.xacro (robot description, xacro)
@@ -1,14 +1,36 @@
 <sdf xmlns:xacro="http://dd">
-    <xacro:include uri="file://data.xacro"/>
-    <xacro:property name="width" value="100"/>
-    <xacro:macro name="m1" params="width bodylen">
-        <collision>
-            <geometry>
-                <cylinder radius="${width}" length="${bodylen}" />
-            </geometry>
-        </collision>
-    </xacro:macro>
-    <xacro:m1 width="${width}" bodylen="10" />
-    <model name="${name}">
+    <xacro:include uri="file://data.xacro" />
+    <xacro:include uri="file://common.xacro" />
+    <xacro:property name="base_mass" value="100" />
+    <model name='heavy_base'>
+        <pose>0 0 0 0 0 0</pose>
+        <link name="heavy_base_link">
+            <!-- position the base such that the bottom touches the floor -->
+            <pose>0 0 0.05 0 0 0</pose>
+            <inertial>
+                <xacro:inertia_box m="100" x="2.2" y="1" z="0.1" />
+            </inertial>
+            <!-- Same geometry as visual -->
+            <collision name="heavy_base_collision">
+                <geometry>
+                    <box>
+                        <size>2.2 1 0.1</size>
+                    </box>
+                </geometry>
+            </collision>
+            <!-- Same geometry as collision -->
+            <visual name="heavy_base_visual">
+                <geometry>
+                    <box>
+                        <size>2.2 1 0.1</size>
+                    </box>
+                </geometry>
+                <material>
+                    <ambient>0 0 1 1</ambient>
+                    <diffuse>0 0 1 1</diffuse>
+                    <specular>0 0 1 1</specular>
+                </material>
+            </visual>
+        </link>
     </model>
 </sdf>

Commit message: added read from xacro:python block

File: examples/py/xacro/source_example/macro.sdf.xacro (robot description, xacro)
@@ -1,7 +1,6 @@
-<sdf version="1.7" xmlns:xacro="http://dd">
+<sdf xmlns:xacro="http://dd">
     <xacro:include uri="file://data.xacro" />
     <xacro:include uri="file://common.xacro" />
-    <xacro:include uri="file://color.xacro" />
-    <xacro:property name="base_mass2" value="100" />
+    <xacro:property name="base_mass" value="100" />
     <model name='heavy_base'>
         <pose>0 0 0 0 0 0</pose>
@@ -10,5 +9,5 @@
             <pose>0 0 0.05 0 0 0</pose>
             <inertial>
-                <xacro:inertia_box m="${base_mass}" x="2.2" y="1" z="0.1" />
+                <xacro:inertia_box m="100" x="2.2" y="1" z="0.1" />
             </inertial>
             <!-- Same geometry as visual -->
@@ -34,19 +33,4 @@
             </visual>
         </link>
-        <link name="wheel_left">
-            <pose>0 -0.5 0 1.5707 0 0</pose>
-            <inertial>
-                <xacro:inertia_cylinder m="${wheel_mass}" r="${wheel_r}" l="${wheel_l}" />
-            </inertial>
-            <visual name="wheel_left_visual">
-                <xacro:geometry_cylinder r="${wheel_r}" l="${wheel_l}"/>
-                <material>
-                    <xacro:color color_name="Red"/>
-                </material>
-            </visual>
-            <collision name="wheel_left_collision">
-                <xacro:geometry_cylinder r="${wheel_r}" l="${wheel_l}"/>
-            </collision>
-        </link>
     </model>
 </sdf>
